Commit message: Creating a map

File: src/docking_description/urdf/docking.xacro (robot description, xacro)
@@ -134,4 +134,32 @@
         <origin xyz="-0.12 0 0.03" />
         <axis xyz="0 0 1" />
+    </joint>
+    <!-- LiDAR -->
+    <link name="lidar_link">
+        <visual>
+            <origin xyz="0 0 0.02" />
+            <geometry>
+                <cylinder radius="0.04" length="0.05" />
+            </geometry>
+            <material name="gray">
+                <color rgba="0.5 0.5 0.5 1" />
+            </material>
+        </visual>
+        <collision>
+            <origin xyz="0 0 0.02" />
+            <geometry>
+                <cylinder radius="0.04" length="0.05" />
+            </geometry>
+        </collision>
+        <inertial>
+            <mass value="0.3" />
+            <origin xyz="0 0 0" />
+            <inertia ixx="0.0005" iyy="0.0005" izz="0.0005" ixy="0" ixz="0" iyz="0" />
+        </inertial>
+    </link>
+    <joint name="lidar_joint" type="fixed">
+        <parent link="base_link" />
+        <child link="lidar_link" />
+        <origin xyz="0 0 0.15" />
     </joint>
     <gazebo>
@@ -157,3 +185,40 @@
         </plugin>
     </gazebo>
+    <gazebo reference="lidar_link">
+        <sensor name="gpu_lidar" type="gpu_lidar">
+            <update_rate>10</update_rate>
+            <topic>scan</topic>
+            <gz_frame_id>lidar_link</gz_frame_id>
+            <frame_id>lidar_link</frame_id>
+            <lidar>
+                <scan>
+                    <horizontal>
+                        <samples>180</samples>
+                        <resolution>1</resolution>
+                        <min_angle>-3.14156</min_angle>
+                        <max_angle>3.14156</max_angle>
+                    </horizontal>
+                </scan>
+                <range>
+                    <min>0.05</min>
+                    <max>10.0</max>
+                    <resolution>0.01</resolution>
+                </range>
+                <noise>
+                    <type>gaussian</type>
+                    <mean>0.0</mean>
+                    <stddev>0.01</stddev>
+                </noise>
+            </lidar>
+            <always_on>1</always_on>
+            <visualize>true</visualize>
+        </sensor>
+    </gazebo>
+    <gazebo>
+        <plugin
+            filename="gz-sim-sensors-system"
+            name="gz::sim::systems::Sensors">
+            <render_engine>ogre2</render_engine>
+        </plugin>
+    </gazebo>
 </robot>

Commit message: Camera Setup

File: src/docking_description/urdf/docking.xacro (robot description, xacro)
@@ -162,4 +162,16 @@
         <child link="lidar_link" />
         <origin xyz="0 0 0.15" />
+    </joint>
+    <link name="camera_link">
+        <visual>
+            <geometry>
+                <box size="0.04 0.04 0.04" />
+            </geometry>
+        </visual>
+    </link>
+    <joint name="camera_joint" type="fixed">
+        <parent link="base_link" />
+        <child link="camera_link" />
+        <origin xyz="0.15 0 0.15" />
     </joint>
     <gazebo>
@@ -215,4 +227,18 @@
         </sensor>
     </gazebo>
+    <gazebo reference="camera_link">
+        <sensor name="camera" type="camera">
+            <update_rate>30</update_rate>
+            <topic>camera/image</topic>
+            <camera>
+                <horizontal_fov>1.396</horizontal_fov>
+                <image>
+                    <width>640</width>
+                    <height>480</height>
+                    <format>R8G8B8</format>
+                </image>
+            </camera>
+        </sensor>
+    </gazebo>
     <gazebo>
         <plugin
